File: kicad/osilloscopen.kicad_pcb (KiCad board)
At the start: 2 copper layers, 28.2 x 34.8 mm, 49 parts, among them J17 OLED, J18 GND, J2 OLED, J3 tip, J4 power, SW1 SW_Push, SW2 SW_Push, SW3 SW_Push, SW4 SW_Push, SW5 POWER, SW6 RESET, U1 AD623AN, U2 ICL7660, U3 STM32F103C6Ux, U4 AP1117-33, U5 XXX, Y1 8MHz

Commit message: layout complete
Parts:
- moved R15 23.4 mm to (239.3, 87.9), turned to 180 degrees
- moved C8 15.1 mm to (251.0, 100.3), turned to -90 degrees
- moved R9 12.5 mm to (231.1, 97.4), turned to 90 degrees
- moved R12 10.5 mm to (244.9, 99.4), turned to 180 degrees
- moved C9 10.4 mm to (240.4, 110.4)
- moved R6 8.39 mm to (232.0, 103.1), turned to 0 degrees
- moved R14 8.35 mm to (241.9, 97.7)
- moved R8 7.37 mm to (232.8, 97.4), turned to -90 degrees
- moved U5 7.12 mm to (240.0, 103.3), turned to 180 degrees
- moved R10 5.83 mm to (245.6, 102.0)
- moved R11 5.46 mm to (244.1, 102.0)
- moved C10 4.96 mm to (235.1, 104.6), turned to 180 degrees
- moved U1 4.62 mm to (237.6, 99.4)
- moved R1 4.39 mm to (227.1, 104.6), turned to 0 degrees
- moved R5 3.97 mm to (232.0, 101.6)
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Connections:
- Y1 pad 2: Net-(C6-Pad2) -> unconnected-(Y1-Pad2)
- Y1 pad 3: (no net) -> Net-(C6-Pad2)
- Y1 pad 4: (no net) -> unconnected-(Y1-Pad4)
Routing:
- net GNDREF: track 0.00 -> 188.0 mm, vias 0 -> 23
- net VDD: track 0.00 -> 94.9 mm, vias 0 -> 4
- net /KEY1: track 0.00 -> 47.6 mm, vias 0 -> 1
- net /KEY4: track 0.00 -> 43.9 mm, vias 0 -> 1
- net /KEY3: track 0.00 -> 37.0 mm, vias 0 -> 1
- net /KEY2: track 0.00 -> 36.2 mm, vias 0 -> 1
- net /SDA: track 0.00 -> 32.2 mm
- net /SCL: track 0.00 -> 31.1 mm
- net /RESET#: track 0.00 -> 30.5 mm, vias 0 -> 1
- net /VDDA: track 0.00 -> 22.3 mm
- net Net-(R12-Pad2): track 0.00 -> 17.1 mm, vias 0 -> 1
- net Net-(C6-Pad2): track 0.00 -> 11.9 mm
- net +5V: track 0.00 -> 11.5 mm
- net Net-(C5-Pad2): track 0.00 -> 11.0 mm
- net -3V3: track 0.00 -> 9.46 mm
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- added copper zone on B.Cu, net GNDREF
- added copper zone on F.Cu, net GNDREF
