File: kicad/osilloscopen.kicad_sch (KiCad schematic)
At the start: 62 parts, among them J1 SWD, J10 Conn_01x01_Male, J11 Conn_01x02_Male, J12 Conn_01x03_Male, J13 Conn_01x02_Male, J14 Conn_01x02_Male, J15 Conn_01x01_Male, J16 Conn_01x03_Male, J17 OLED, J18 GND, J19 VBAT, J2 OLED, J3 tip, J4 power, J5 Conn_01x03_Male, J6 Conn_01x01_Male, J7 Conn_01x04_Male, J8 Conn_01x01_Male, J9 Conn_01x03_Male, SW1 SW_Push, SW2 SW_Push, SW3 SW_Push, SW4 SW_Push, SW5 POWER, SW6 RESET, U1 AD623AN, U2 ICL7660, U3 STM32F103C6Ux, U4 AP1117-33, U5 XXX, Y1 8MHz

Commit message: layout complete
Parts:
- Y1: symbol Device:Crystal -> Device:Crystal_GND24_Small
Connections:
- net at C6.2, R13.2, U3.6 (PD1): now also Y1.3; no longer Y1.2
